File: RP2040-Neopixel-Strip-Driver/RP2040.kicad_sch (KiCad schematic)
At the start: 37 parts, among them J201 TYPE-C-31-M-12, J202 Conn_01x03, SW202 ~{USB_BOOT}, U201 AZ1117R-3.3TRE1, U202 RP2040, U205 W25Q128JVS, Y201 Crystal_GND24

Commit message: Continued to shrink PCB, replaced regulator and mem with smaller ICs, removed 1206 caps
Parts:
- removed C209, C210: 100uF, Capacitor_SMD:C_1206_3216Metric, symbol Device:C_Small
- J203: value (none) -> NeopixelStrip; footprint (none) -> Breadstick Footprints:NeopixelStrip
- U201: value AZ1117R-3.3TRE1 -> XC6206P332MR; footprint Package_TO_SOT_SMD:SOT-89-3 -> Package_TO_SOT_SMD:SOT-23; JLCPCB P/N C108493 -> C5446
- U205: value W25Q128JVS -> W25Q128JVPIQ; footprint Package_SO:SOIC-8_5.23x5.23mm_P1.27mm -> Package_SON:WSON-8-1EP_6x5mm_P1.27mm_EP3.4x4.3mm; JLCPCB P/N C97521 -> C190862
Connections:
- net GND: now also U205.9 (PAD)
Changed lines of the file:
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@@
   (junction (at 60.96 54.61) (diameter 0) (color 0 0 0 0)
   )
-  (junction (at 153.67 173.99) (diameter 0) (color 0 0 0 0)
-  )
   (junction (at 43.18 77.47) (diameter 0) (color 0 0 0 0)
   )
@@
   (junction (at 119.38 30.48) (diameter 0) (color 0 0 0 0)
   )
+  (junction (at 251.46 153.67) (diameter 0) (color 0 0 0 0)
+  )
   (junction (at 148.59 173.99) (diameter 0) (color 0 0 0 0)
   )
@@
   (junction (at 119.38 41.91) (diameter 0) (color 0 0 0 0)
   )
-  (junction (at 111.76 173.99) (diameter 0) (color 0 0 0 0)
-  )
   (junction (at 62.23 40.64) (diameter 0) (color 0 0 0 0)
   )
@@
     (stroke (width 0) (type default) (color 0 0 0 0))
   )
-  (wire (pts (xy 153.67 173.99) (xy 161.29 173.99))
+  (wire (pts (xy 148.59 173.99) (xy 161.29 173.99))
     (stroke (width 0) (type default) (color 0 0 0 0))
   )
@@
     (stroke (width 0) (type default) (color 0 0 0 0))
   )
-  (wire (pts (xy 148.59 173.99) (xy 153.67 173.99))
-    (stroke (width 0) (type default) (color 0 0 0 0))
-  )
   (wire (pts (xy 111.76 130.81) (xy 111.76 133.35))
     (stroke (width 0) (type default) (color 0 0 0 0))
@@
     (stroke (width 0) (type default) (color 0 0 0 0))
   )
-  (wire (pts (xy 111.76 173.99) (xy 116.84 173.99))
+  (wire (pts (xy 102.87 173.99) (xy 116.84 173.99))
     (stroke (width 0) (type default) (color 0 0 0 0))
   )
@@
     (stroke (width 0) (type default) (color 0 0 0 0))
   )
-  (wire (pts (xy 102.87 173.99) (xy 111.76 173.99))
-    (stroke (width 0) (type default) (color 0 0 0 0))
-  )
   (wire (pts (xy 134.62 77.47) (xy 140.97 77.47))
     (stroke (width 0) (type default) (color 0 0 0 0))
@@
   )
   (wire (pts (xy 43.18 77.47) (xy 43.18 81.28))
+    (stroke (width 0) (type default) (color 0 0 0 0))
+  )
+  (wire (pts (xy 251.46 153.67) (xy 255.27 153.67))
     (stroke (width 0) (type default) (color 0 0 0 0))
   )
@@
     )
   )
-  (symbol (lib_id "Device:C_Small") (at 111.76 176.53 0) (unit 1)
-    (in_bom yes) (on_board yes)
-    (property "Reference" "C209" (id 0) (at 104.14 176.53 0)
-      (effects (font (size 1.27 1.27)) (justify left))
-    )
-    (property "Value" "100uF" (id 1) (at 104.14 179.07 0)
-      (effects (font (size 1.27 1.27)) (justify left))
-    )
-    (property "Footprint" "Capacitor_SMD:C_1206_3216Metric" (id 2) (at 111.76 176.53 0)
-      (effects (font (size 1.27 1.27)) hide)
-    )
-    (property "Datasheet" "~" (id 3) (at 111.76 176.53 0)
-      (effects (font (size 1.27 1.27)) hide)
-    )
-    (property "JLCPCB P/N" "C15008" (id 4) (at 111.76 176.53 0)
-      (effects (font (size 1.27 1.27)) hide)
-    )
-    (pin "1")
-    (pin "2")
-  )
   (symbol (lib_id "BreadstickLibrary:AZ1117R-3.3TRE1") (at 132.08 175.26 0) (unit 1)
     (in_bom yes) (on_board yes) (fields_autoplaced)
     (property "Reference" "U201" (id 0) (at 132.715 167.64 0))
-    (property "Value" "AZ1117R-3.3TRE1" (id 1) (at 132.715 170.18 0))
-    (property "Footprint" "Package_TO_SOT_SMD:SOT-89-3" (id 2) (at 132.08 175.26 0)
+    (property "Value" "XC6206P332MR" (id 1) (at 132.715 170.18 0))
+    (property "Footprint" "Package_TO_SOT_SMD:SOT-23" (id 2) (at 132.08 175.26 0)
       (effects (font (size 1.27 1.27)) hide)
     )
@@
       (effects (font (size 1.27 1.27)) hide)
     )
-    (property "JLCPCB P/N" "C108493" (id 4) (at 132.08 175.26 0)
+    (property "JLCPCB P/N" "C5446" (id 4) (at 132.08 175.26 0)
       (effects (font (size 1.27 1.27)) hide)
     )
@@
     )
     (pin "1")
-  )
-  (symbol (lib_id "Device:C_Small") (at 153.67 176.53 0) (unit 1)
-    (in_bom yes) (on_board yes)
-    (property "Reference" "C210" (id 0) (at 156.21 176.53 0)
-      (effects (font (size 1.27 1.27)) (justify left))
-    )
-    (property "Value" "100uF" (id 1) (at 156.21 179.07 0)
-      (effects (font (size 1.27 1.27)) (justify left))
-    )
-    (property "Footprint" "Capacitor_SMD:C_1206_3216Metric" (id 2) (at 153.67 176.53 0)
-      (effects (font (size 1.27 1.27)) hide)
-    )
-    (property "Datasheet" "~" (id 3) (at 153.67 176.53 0)
-      (effects (font (size 1.27 1.27)) hide)
-    )
-    (property "JLCPCB P/N" "C15008" (id 4) (at 153.67 176.53 0)
-      (effects (font (size 1.27 1.27)) hide)
-    )
-    (pin "1")
-    (pin "2")
   )
   (symbol (lib_id "Device:C_Small") (at 40.64 43.18 0) (unit 1)
@@
     (pin "9")
   )
-  (symbol (lib_id "power:GND") (at 153.67 179.07 0) (unit 1)
-    (in_bom yes) (on_board yes)
-    (property "Reference" "#PWR0214" (id 0) (at 153.67 185.42 0)
-      (effects (font (size 1.27 1.27)) hide)
-    )
-    (property "Value" "GND" (id 1) (at 153.67 182.88 0))
-    (property "Footprint" "" (id 2) (at 153.67 179.07 0)
-      (effects (font (size 1.27 1.27)) hide)
-    )
-    (property "Datasheet" "" (id 3) (at 153.67 179.07 0)
-      (effects (font (size 1.27 1.27)) hide)
-    )
-    (pin "1")
-  )
   (symbol (lib_id "Memory_Flash:W25Q128JVS") (at 251.46 143.51 0) (unit 1)
     (in_bom yes) (on_board yes) (fields_autoplaced)
@@
       (effects (font (size 1.27 1.27)) (justify left))
     )
-    (property "Value" "W25Q128JVS" (id 1) (at 253.4794 133.35 0)
-      (effects (font (size 1.27 1.27)) (justify left))
-    )
-    (property "Footprint" "Package_SO:SOIC-8_5.23x5.23mm_P1.27mm" (id 2) (at 251.46 143.51 0)
+    (property "Value" "W25Q128JVPIQ" (id 1) (at 253.4794 133.35 0)
+      (effects (font (size 1.27 1.27)) (justify left))
+    )
+    (property "Footprint" "Package_SON:WSON-8-1EP_6x5mm_P1.27mm_EP3.4x4.3mm" (id 2) (at 251.46 143.51 0)
       (effects (font (size 1.27 1.27)) hide)
     )
@@
       (effects (font (size 1.27 1.27)) hide)
     )
-    (property "JLCPCB P/N" "C97521" (id 4) (at 251.46 143.51 0)
+    (property "JLCPCB P/N" "C190862" (id 4) (at 251.46 143.51 0)
       (effects (font (size 1.27 1.27)) hide)
     )
@@
     (pin "7")
     (pin "8")
+    (pin "9")
   )
   (symbol (lib_id "Device:R") (at 219.71 78.74 90) (unit 1)
@@
       (effects (font (size 1.27 1.27)) (justify left))
     )
-    (property "Value" "" (id 1) (at 55.88 189.2299 0)
-      (effects (font (size 1.27 1.27)) (justify left))
-    )
-    (property "Footprint" "" (id 2) (at 53.34 187.96 0)
+    (property "Value" "NeopixelStrip" (id 1) (at 55.88 189.2299 0)
+      (effects (font (size 1.27 1.27)) (justify left))
+    )
+    (property "Footprint" "Breadstick Footprints:NeopixelStrip" (id 2) (at 53.34 187.96 0)
       (effects (font (size 1.27 1.27)) hide)
     )
@@
       (effects (font (size 1.27 1.27)) hide)
     )
-    (pin "1")
-  )
-  (symbol (lib_id "power:GND") (at 111.76 179.07 0) (unit 1)
-    (in_bom yes) (on_board yes)
-    (property "Reference" "#PWR0201" (id 0) (at 111.76 185.42 0)
-      (effects (font (size 1.27 1.27)) hide)
-    )
-    (property "Value" "GND" (id 1) (at 111.76 182.88 0))
-    (property "Footprint" "" (id 2) (at 111.76 179.07 0)
-      (effects (font (size 1.27 1.27)) hide)
-    )
-    (property "Datasheet" "" (id 3) (at 111.76 179.07 0)
-      (effects (font (size 1.27 1.27)) hide)
-    )

Commit message: Continued to shrink board.
Parts:
- removed C207: 10uF, Breadstick Footprints:Perfect_0402_Cap, symbol Device:C_Small
Other:
- note added: "Placed close to uC decoupling caps."
Changed lines of the file:
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@@
+    (effects (font (size 1.27 1.27)) (justify left bottom))
+  )
+  (text "Placed close to uC decoupling caps." (at 139.7 179.07 0)
     (effects (font (size 1.27 1.27)) (justify left bottom))
   )
@@
     (pin "1")
   )
-  (symbol (lib_id "Device:C_Small") (at 148.59 176.53 0) (unit 1)
-    (in_bom yes) (on_board yes)
-    (property "Reference" "C207" (id 0) (at 140.97 176.53 0)
-      (effects (font (size 1.27 1.27)) (justify left))
-    )
-    (property "Value" "10uF" (id 1) (at 140.97 179.07 0)
-      (effects (font (size 1.27 1.27)) (justify left))
-    )
-    (property "Footprint" "Breadstick Footprints:Perfect_0402_Cap" (id 2) (at 148.59 176.53 0)
-      (effects (font (size 1.27 1.27)) hide)
-    )
-    (property "Datasheet" "~" (id 3) (at 148.59 176.53 0)
-      (effects (font (size 1.27 1.27)) hide)
-    )
-    (property "JLCPCB P/N" "C15525" (id 4) (at 148.59 176.53 0)
-      (effects (font (size 1.27 1.27)) hide)
-    )
-    (pin "1")
-    (pin "2")
-  )
   (symbol (lib_id "power:GND") (at 226.06 34.29 0) (unit 1)
     (in_bom yes) (on_board yes)
@@
     (pin "2")
   )
-  (symbol (lib_id "power:GND") (at 148.59 179.07 0) (unit 1)
-    (in_bom yes) (on_board yes)
-    (property "Reference" "#PWR0210" (id 0) (at 148.59 185.42 0)
-      (effects (font (size 1.27 1.27)) hide)
-    )
-    (property "Value" "GND" (id 1) (at 148.59 182.88 0))
-    (property "Footprint" "" (id 2) (at 148.59 179.07 0)
-      (effects (font (size 1.27 1.27)) hide)
-    )
-    (property "Datasheet" "" (id 3) (at 148.59 179.07 0)
-      (effects (font (size 1.27 1.27)) hide)
-    )
-    (pin "1")
-  )
   (symbol (lib_id "Device:C_Small") (at 29.21 43.18 0) (unit 1)

Commit message: Added bulk decoupling capacitors and PTC resetable fuse, planning level shifter.
Parts:
- added C207: (no value), symbol Device:C_Small
- added C209: 220uF, Capacitor_SMD:C_1210_3225Metric, symbol Device:C_Small
- added F201: (no value), symbol Device:Polyfuse
- added J204: (no value), symbol Connector_Generic:Conn_01x01
- added J205, J206: (no value), Connector_PinSocket_2.54mm:PinSocket_1x01_P2.54mm_Vertical, symbol Connector_Generic:Conn_01x01
Connections:
- net VHI is gone; now on net VBUS: C201.1, U201.3 (IN)
- net GND: now also C207.2, C209.2, J206.1 (Pin_1)
- net VBUS: now also C207.1, C209.1, F201.1, J204.1 (Pin_1); no longer D203.2 (A2), D205.2 (A2), J201.A4B9 (VBUS), J201.B4A9 (VBUS)
- new net: D203.2 (A2), D205.2 (A2), F201.2, J201.A4B9 (VBUS), J201.B4A9 (VBUS)
Other:
- moved on the sheet: D201, D202, D203, D205, J201, R212, R214

Commit message: Worked on layout, still selecting a level shifter.
Parts:
- C207: value (none) -> 220uF; footprint (none) -> Capacitor_SMD:C_1210_3225Metric
- F201: value (none) -> 1.5A, 3A Trip; footprint (none) -> Resistor_SMD:R_0805_2012Metric
- J204: value (none) -> 5V; footprint (none) -> Connector_PinSocket_2.54mm:PinSocket_1x01_P2.54mm_Vertical
- J205: value (none) -> TO BE DECIDED
- J206: value (none) -> GND
Other:
- note added: "Level Shifter Candidate: NLSX4302EBMUTCG C893527"
- moved on the sheet: C207, C209
Changed lines of the file:
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@@
   (junction (at 60.96 54.61) (diameter 0) (color 0 0 0 0)
   )
-  (junction (at 41.91 213.36) (diameter 0) (color 0 0 0 0)
-  )
-  (junction (at 44.45 205.74) (diameter 0) (color 0 0 0 0)
+  (junction (at 179.07 146.05) (diameter 0) (color 0 0 0 0)
+  )
+  (junction (at 181.61 138.43) (diameter 0) (color 0 0 0 0)
   )
   (junction (at 43.18 77.47) (diameter 0) (color 0 0 0 0)
@@
   (junction (at 234.95 140.97) (diameter 0) (color 0 0 0 0)
   )
-  (wire (pts (xy 35.56 207.01) (xy 35.56 205.74))
-    (stroke (width 0) (type default) (color 0 0 0 0))
-  )
-  (wire (pts (xy 35.56 212.09) (xy 35.56 213.36))
+  (wire (pts (xy 172.72 139.7) (xy 172.72 138.43))
+    (stroke (width 0) (type default) (color 0 0 0 0))
+  )
+  (wire (pts (xy 172.72 144.78) (xy 172.72 146.05))
     (stroke (width 0) (type default) (color 0 0 0 0))
   )
@@
     (stroke (width 0) (type default) (color 0 0 0 0))
   )
-  (wire (pts (xy 44.45 205.74) (xy 46.99 205.74))
+  (wire (pts (xy 181.61 138.43) (xy 184.15 138.43))
     (stroke (width 0) (type default) (color 0 0 0 0))
   )
@@
     (stroke (width 0) (type default) (color 0 0 0 0))
   )
-  (wire (pts (xy 35.56 213.36) (xy 41.91 213.36))
+  (wire (pts (xy 172.72 146.05) (xy 179.07 146.05))
     (stroke (width 0) (type default) (color 0 0 0 0))
   )
@@
     (stroke (width 0) (type default) (color 0 0 0 0))
   )
-  (wire (pts (xy 43.18 203.2) (xy 44.45 203.2))
+  (wire (pts (xy 180.34 135.89) (xy 181.61 135.89))
     (stroke (width 0) (type default) (color 0 0 0 0))
   )
@@
     (stroke (width 0) (type default) (color 0 0 0 0))
   )
-  (wire (pts (xy 46.99 212.09) (xy 46.99 213.36))
+  (wire (pts (xy 184.15 144.78) (xy 184.15 146.05))
     (stroke (width 0) (type default) (color 0 0 0 0))
   )
@@
     (stroke (width 0) (type default) (color 0 0 0 0))
   )
-  (wire (pts (xy 35.56 205.74) (xy 44.45 205.74))
+  (wire (pts (xy 172.72 138.43) (xy 181.61 138.43))
     (stroke (width 0) (type default) (color 0 0 0 0))
   )
@@
     (stroke (width 0) (type default) (color 0 0 0 0))
   )
-  (wire (pts (xy 44.45 203.2) (xy 44.45 205.74))
+  (wire (pts (xy 181.61 135.89) (xy 181.61 138.43))
     (stroke (width 0) (type default) (color 0 0 0 0))
   )
@@
     (stroke (width 0) (type default) (color 0 0 0 0))
   )
-  (wire (pts (xy 41.91 213.36) (xy 46.99 213.36))
+  (wire (pts (xy 179.07 146.05) (xy 184.15 146.05))
     (stroke (width 0) (type default) (color 0 0 0 0))
   )
@@
     (stroke (width 0) (type default) (color 0 0 0 0))
   )
-  (wire (pts (xy 46.99 205.74) (xy 46.99 207.01))
+  (wire (pts (xy 184.15 138.43) (xy 184.15 139.7))
     (stroke (width 0) (type default) (color 0 0 0 0))
   )
@@
   )
   (text "ESD Protection" (at 203.2 17.78 0)
+    (effects (font (size 1.27 1.27)) (justify left bottom))
+  )
+  (text "Level Shifter Candidate:\nNLSX4302EBMUTCG\nC893527" (at 96.52 153.67 0)
     (effects (font (size 1.27 1.27)) (justify left bottom))
   )
@@
     )
   )
-  (global_label "VBUS" (shape input) (at 43.18 203.2 180) (fields_autoplaced)
-    (effects (font (size 1.27 1.27)) (justify right))
-    (property "Intersheet References" "${INTERSHEET_REFS}" (id 0) (at 35.8683 203.2794 0)
+  (global_label "VBUS" (shape input) (at 180.34 135.89 180) (fields_autoplaced)
+    (effects (font (size 1.27 1.27)) (justify right))
+    (property "Intersheet References" "${INTERSHEET_REFS}" (id 0) (at 173.0283 135.9694 0)
       (effects (font (size 1.27 1.27)) (justify right) hide)
     )
@@
       (effects (font (size 1.27 1.27)) (justify left))
     )
-    (property "Value" "" (id 1) (at 60.96 151.13 0)
-      (effects (font (size 1.27 1.27)) (justify left))
-    )
-    (property "Footprint" "" (id 2) (at 53.34 151.13 0)
+    (property "Value" "5V" (id 1) (at 60.96 151.13 0)
+      (effects (font (size 1.27 1.27)) (justify left))
+    )
+    (property "Footprint" "Connector_PinSocket_2.54mm:PinSocket_1x01_P2.54mm_Vertical" (id 2) (at 53.34 151.13 0)
       (effects (font (size 1.27 1.27)) hide)
     )
@@
       (effects (font (size 1.27 1.27)) (justify left))
     )
-    (property "Value" "" (id 1) (at 60.96 154.94 0)
+    (property "Value" "TO BE DECIDED" (id 1) (at 60.96 154.94 0)
       (effects (font (size 1.27 1.27)) (justify left))
     )
@@
       (effects (font (size 1.27 1.27)) (justify left))
     )
-    (property "Value" "" (id 1) (at 60.96 158.75 0)
+    (property "Value" "GND" (id 1) (at 60.96 158.75 0)
       (effects (font (size 1.27 1.27)) (justify left))
     )
@@
     (pin "1")
   )
-  (symbol (lib_id "Device:C_Small") (at 35.56 209.55 0) (unit 1)
-    (in_bom yes) (on_board yes)
-    (property "Reference" "C207" (id 0) (at 38.1 208.28 0)
-      (effects (font (size 1.27 1.27)) (justify left))
-    )
-    (property "Value" "" (id 1) (at 38.1 210.82 0)
-      (effects (font (size 1.27 1.27)) (justify left))
-    )
-    (property "Footprint" "" (id 2) (at 35.56 209.55 0)
-      (effects (font (size 1.27 1.27)) hide)
-    )
-    (property "Datasheet" "~" (id 3) (at 35.56 209.55 0)
-      (effects (font (size 1.27 1.27)) hide)
-    )
-    (property "JLCPCB P/N" "C400951" (id 4) (at 35.56 209.55 0)
+  (symbol (lib_id "Device:C_Small") (at 172.72 142.24 0) (unit 1)
+    (in_bom yes) (on_board yes)
+    (property "Reference" "C207" (id 0) (at 175.26 140.97 0)
+      (effects (font (size 1.27 1.27)) (justify left))
+    )
+    (property "Value" "220uF" (id 1) (at 175.26 143.51 0)
+      (effects (font (size 1.27 1.27)) (justify left))
+    )
+    (property "Footprint" "Capacitor_SMD:C_1210_3225Metric" (id 2) (at 172.72 142.24 0)
+      (effects (font (size 1.27 1.27)) hide)
+    )
+    (property "Datasheet" "~" (id 3) (at 172.72 142.24 0)
+      (effects (font (size 1.27 1.27)) hide)
+    )
+    (property "JLCPCB P/N" "C400951" (id 4) (at 172.72 142.24 0)
       (effects (font (size 1.27 1.27)) hide)
     )
@@
     (pin "9")
   )
-  (symbol (lib_id "power:GND") (at 41.91 213.36 0) (unit 1)
-    (in_bom yes) (on_board yes)
-    (property "Reference" "#PWR0210" (id 0) (at 41.91 219.71 0)
-      (effects (font (size 1.27 1.27)) hide)
-    )
-    (property "Value" "GND" (id 1) (at 41.91 217.17 0))
-    (property "Footprint" "" (id 2) (at 41.91 213.36 0)
-      (effects (font (size 1.27 1.27)) hide)
-    )
-    (property "Datasheet" "" (id 3) (at 41.91 213.36 0)
+  (symbol (lib_id "power:GND") (at 179.07 146.05 0) (unit 1)
+    (in_bom yes) (on_board yes)
+    (property "Reference" "#PWR0210" (id 0) (at 179.07 152.4 0)
+      (effects (font (size 1.27 1.27)) hide)
+    )
+    (property "Value" "GND" (id 1) (at 179.07 149.86 0))
+    (property "Footprint" "" (id 2) (at 179.07 146.05 0)
+      (effects (font (size 1.27 1.27)) hide)
+    )
+    (property "Datasheet" "" (id 3) (at 179.07 146.05 0)
       (effects (font (size 1.27 1.27)) hide)
     )
@@
     (in_bom yes) (on_board yes)
     (property "Reference" "F201" (id 0) (at 251.46 73.66 90))
-    (property "Value" "" (id 1) (at 256.54 78.74 90))
-    (property "Footprint" "" (id 2) (at 246.38 77.47 0)
+    (property "Value" "1.5A, 3A Trip" (id 1) (at 256.54 78.74 90))
+    (property "Footprint" "Resistor_SMD:R_0805_2012Metric" (id 2) (at 246.38 77.47 0)
       (effects (font (size 1.27 1.27)) (justify left) hide)
     )
@@
     (pin "2")
   )
-  (symbol (lib_id "Device:C_Small") (at 46.99 209.55 0) (unit 1)
-    (in_bom yes) (on_board yes)
-    (property "Reference" "C209" (id 0) (at 49.53 208.28 0)
-      (effects (font (size 1.27 1.27)) (justify left))
-    )
-    (property "Value" "220uF" (id 1) (at 49.53 210.82 0)
-      (effects (font (size 1.27 1.27)) (justify left))
-    )
-    (property "Footprint" "Capacitor_SMD:C_1210_3225Metric" (id 2) (at 46.99 209.55 0)
-      (effects (font (size 1.27 1.27)) hide)
-    )
-    (property "Datasheet" "~" (id 3) (at 46.99 209.55 0)
-      (effects (font (size 1.27 1.27)) hide)
-    )
-    (property "JLCPCB P/N" "C400951" (id 4) (at 46.99 209.55 0)
-      (effects (font (size 1.27 1.27)) hide)
-    )
+  (symbol (lib_id "Device:C_Small") (at 184.15 142.24 0) (unit 1)
+    (in_bom yes) (on_board yes)
+    (property "Reference" "C209" (id 0) (at 186.69 140.97 0)
+      (effects (font (size 1.27 1.27)) (justify left))
+    )
+    (property "Value" "220uF" (id 1) (at 186.69 143.51 0)
+      (effects (font (size 1.27 1.27)) (justify left))
+    )
+    (property "Footprint" "Capacitor_SMD:C_1210_3225Metric" (id 2) (at 184.15 142.24 0)
+      (effects (font (size 1.27 1.27)) hide)
+    )
+    (property "Datasheet" "~" (id 3) (at 184.15 142.24 0)
+      (effects (font (size 1.27 1.27)) hide)
+    )
+    (property "JLCPCB P/N" "C400951" (id 4) (at 184.15 142.24 0)
+      (effects (font (size 1.27 1.27)) hide)
+    )

Commit message: Moved USB and 3.3V Regulator from RP2040 to Power Sheet
Parts:
- removed C201: 10uF, Breadstick Footprints:Perfect_0402_Cap, symbol Device:C_Small
- removed D203, D205: ESD_TVS, Breadstick Footprints:Perfect_0402_Resistor, symbol Device:D_TVS_Filled
- removed F201: 1.5A, 3A Trip, Resistor_SMD:R_0805_2012Metric, symbol Device:Polyfuse
- removed J201: TYPE-C-31-M-12, TYPE-C-31-M-12:HRO_TYPE-C-31-M-12, symbol TYPE-C-31-M-12:TYPE-C-31-M-12
- removed R212, R214: 5k1, Breadstick Footprints:Perfect_0402_Resistor, symbol Device:R
- removed U201: XC6206P332MR, Package_TO_SOT_SMD:SOT-23, symbol BreadstickLibrary:AZ1117R-3.3TRE1
Other:
- note added: "USB Connector On Power Sheet"
- note removed: "Placed close to uC decoupling caps."
- note removed: "USB-C"
