File: RP2040-Neopixel-Strip-Driver/RP2040.kicad_sch (KiCad schematic)
At the start: 32 parts, among them J202 Conn_01x03, J203 NeopixelStrip, J204 5V, J205 TO BE DECIDED, J206 GND, SW202 ~{USB_BOOT}, U202 RP2040, U205 W25Q128JVPIQ, Y201 Crystal_GND24

Commit message: Reworked the USB-C Connector Symbol to clean up schematic
Parts:
- removed D201, D202: ESD_TVS, Breadstick Footprints:Perfect_0402_Resistor, symbol Device:D_TVS_Filled
Other:
- note removed: "ESD Protection"
Changed lines of the file:
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@@
-    (stroke (width 0) (type default) (color 0 0 0 0))
-  )
-  (polyline (pts (xy 204.47 17.78) (xy 204.47 43.18))
     (stroke (width 0) (type default) (color 0 0 0 0))
   )
@@
     (stroke (width 0) (type default) (color 0 0 0 0))
   )
-  (polyline (pts (xy 204.47 17.78) (xy 261.62 17.78))
-    (stroke (width 0) (type default) (color 0 0 0 0))
-  )
   (wire (pts (xy 234.95 124.46) (xy 246.38 124.46))
     (stroke (width 0) (type default) (color 0 0 0 0))
@@
     (stroke (width 0) (type default) (color 0 0 0 0))
   )
-  (polyline (pts (xy 204.47 43.18) (xy 261.62 43.18))
-    (stroke (width 0) (type default) (color 0 0 0 0))
-  )
   (wire (pts (xy 31.75 77.47) (xy 31.75 71.12))
     (stroke (width 0) (type default) (color 0 0 0 0))
@@
     (stroke (width 0) (type default) (color 0 0 0 0))
   )
-  (polyline (pts (xy 261.62 43.18) (xy 261.62 17.78))
-    (stroke (width 0) (type default) (color 0 0 0 0))
-  )
   (wire (pts (xy 63.5 59.69) (xy 63.5 62.23))
     (stroke (width 0) (type default) (color 0 0 0 0))
@@
     (effects (font (size 1.27 1.27)) (justify left bottom))
   )
-  (text "ESD Protection" (at 203.2 17.78 0)
-    (effects (font (size 1.27 1.27)) (justify left bottom))
-  )
   (text "Level Shifter Candidate:\nNLSX4302EBMUTCG\nC893527" (at 96.52 153.67 0)
     (effects (font (size 1.27 1.27)) (justify left bottom))
@@
   (text "Do Not Use GPIO15 Errata RP2040-E5" (at 110.49 85.09 0)
     (effects (font (size 1.27 1.27)) (justify left bottom))
-  )
-  (label "USB_D-" (at 246.38 25.4 180)
-    (effects (font (size 1.27 1.27)) (justify right bottom))
   )
   (label "MCU_QSPI_SD2" (at 109.22 67.31 0)
@@
   (label "MCU_USB_D+" (at 113.03 80.01 0)
     (effects (font (size 1.27 1.27)) (justify left bottom))
-  )
-  (label "USB_D+" (at 227.33 25.4 180)
-    (effects (font (size 1.27 1.27)) (justify right bottom))
   )
   (label "MCU_QSPI_CSN" (at 233.68 140.97 180)
@@
     )
     (property "Datasheet" "" (id 3) (at 204.47 151.13 0)
-      (effects (font (size 1.27 1.27)) hide)
-    )
-    (pin "1")
-  )
-  (symbol (lib_id "power:GND") (at 246.38 33.02 0) (unit 1)
-    (in_bom yes) (on_board yes)
-    (property "Reference" "#PWR0103" (id 0) (at 246.38 39.37 0)
-      (effects (font (size 1.27 1.27)) hide)
-    )
-    (property "Value" "GND" (id 1) (at 246.38 36.83 0))
-    (property "Footprint" "" (id 2) (at 246.38 33.02 0)
-      (effects (font (size 1.27 1.27)) hide)
-    )
-    (property "Datasheet" "" (id 3) (at 246.38 33.02 0)
       (effects (font (size 1.27 1.27)) hide)
     )
@@
     (pin "2")
   )
-  (symbol (lib_id "Device:D_TVS_Filled") (at 246.38 29.21 90) (unit 1)
-    (in_bom yes) (on_board yes)
-    (property "Reference" "D202" (id 0) (at 248.92 27.9399 90)
-      (effects (font (size 1.27 1.27)) (justify right))
-    )
-    (property "Value" "ESD_TVS" (id 1) (at 248.92 30.4799 90)
-      (effects (font (size 1.27 1.27)) (justify right))
-    )
-    (property "Footprint" "Breadstick Footprints:Perfect_0402_Resistor" (id 2) (at 246.38 29.21 0)
-      (effects (font (size 1.27 1.27)) hide)
-    )
-    (property "Datasheet" "~" (id 3) (at 246.38 29.21 0)
-      (effects (font (size 1.27 1.27)) hide)
-    )
-    (property "JLCPCB P/N" "C316049" (id 4) (at 246.38 29.21 0)
-      (effects (font (size 1.27 1.27)) hide)
-    )
-    (pin "1")
-    (pin "2")
-  )
   (symbol (lib_id "power:GND") (at 40.64 45.72 0) (unit 1)
     (in_bom yes) (on_board yes)
@@
     )
     (property "Datasheet" "" (id 3) (at 38.1 59.69 0)
-      (effects (font (size 1.27 1.27)) hide)
-    )
-    (pin "1")
-  )
-  (symbol (lib_id "power:GND") (at 227.33 33.02 0) (unit 1)
-    (in_bom yes) (on_board yes)
-    (property "Reference" "#PWR0243" (id 0) (at 227.33 39.37 0)
-      (effects (font (size 1.27 1.27)) hide)
-    )
-    (property "Value" "GND" (id 1) (at 227.33 36.83 0))
-    (property "Footprint" "" (id 2) (at 227.33 33.02 0)
-      (effects (font (size 1.27 1.27)) hide)
-    )
-    (property "Datasheet" "" (id 3) (at 227.33 33.02 0)
       (effects (font (size 1.27 1.27)) hide)
     )
@@
       (effects (font (size 1.27 1.27)) hide)
     )
-    (pin "1")
-    (pin "2")
-  )
-  (symbol (lib_id "Device:D_TVS_Filled") (at 227.33 29.21 90) (unit 1)
-    (in_bom yes) (on_board yes) (fields_autoplaced)
-    (property "Reference" "D201" (id 0) (at 229.87 27.9399 90)
-      (effects (font (size 1.27 1.27)) (justify right))
-    )
-    (property "Value" "ESD_TVS" (id 1) (at 229.87 30.4799 90)
-      (effects (font (size 1.27 1.27)) (justify right))
-    )
-    (property "Footprint" "Breadstick Footprints:Perfect_0402_Resistor" (id 2) (at 227.33 29.21 0)
-      (effects (font (size 1.27 1.27)) hide)
-    )
-    (property "Datasheet" "~" (id 3) (at 227.33 29.21 0)
-      (effects (font (size 1.27 1.27)) hide)
-    )
-    (property "JLCPCB P/N" "C316049" (id 4) (at 227.33 29.21 0)
-      (effects (font (size 1.27 1.27)) hide)
-    )

Commit message: Removed unnecessary pwr and gnd pins, moved decoupling caps to power sheet
Parts:
- removed C207, C209: 220uF, Capacitor_SMD:C_1210_3225Metric, symbol Device:C_Small
- removed J204: 5V, Connector_PinSocket_2.54mm:PinSocket_1x01_P2.54mm_Vertical, symbol Connector_Generic:Conn_01x01
- removed J205: TO BE DECIDED, Connector_PinSocket_2.54mm:PinSocket_1x01_P2.54mm_Vertical, symbol Connector_Generic:Conn_01x01
- removed J206: GND, Connector_PinSocket_2.54mm:PinSocket_1x01_P2.54mm_Vertical, symbol Connector_Generic:Conn_01x01
Other:
- note removed: "LDO"
- note removed: "Level Shifter Candidate: NLSX4302EBMUTCG C893527"
Changed lines of the file:
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@@
   (junction (at 60.96 54.61) (diameter 0) (color 0 0 0 0)
   )
-  (junction (at 179.07 146.05) (diameter 0) (color 0 0 0 0)
-  )
-  (junction (at 181.61 138.43) (diameter 0) (color 0 0 0 0)
-  )
   (junction (at 43.18 77.47) (diameter 0) (color 0 0 0 0)
   )
@@
   (junction (at 234.95 140.97) (diameter 0) (color 0 0 0 0)
   )
-  (wire (pts (xy 172.72 139.7) (xy 172.72 138.43))
-    (stroke (width 0) (type default) (color 0 0 0 0))
-  )
-  (wire (pts (xy 172.72 144.78) (xy 172.72 146.05))
-    (stroke (width 0) (type default) (color 0 0 0 0))
-  )
   (polyline (pts (xy 15.24 144.78) (xy 157.48 144.78))
     (stroke (width 0) (type default) (color 0 0 0 0))
   )
-  (wire (pts (xy 181.61 138.43) (xy 184.15 138.43))
-    (stroke (width 0) (type default) (color 0 0 0 0))
-  )
   (wire (pts (xy 49.53 74.93) (xy 63.5 74.93))
     (stroke (width 0) (type default) (color 0 0 0 0))
@@
     (stroke (width 0) (type default) (color 0 0 0 0))
   )
-  (wire (pts (xy 172.72 146.05) (xy 179.07 146.05))
-    (stroke (width 0) (type default) (color 0 0 0 0))
-  )
   (wire (pts (xy 60.96 54.61) (xy 63.5 54.61))
     (stroke (width 0) (type default) (color 0 0 0 0))
@@
     (stroke (width 0) (type default) (color 0 0 0 0))
   )
-  (wire (pts (xy 180.34 135.89) (xy 181.61 135.89))
-    (stroke (width 0) (type default) (color 0 0 0 0))
-  )
   (wire (pts (xy 110.49 41.91) (xy 110.49 30.48))
     (stroke (width 0) (type default) (color 0 0 0 0))
@@
     (stroke (width 0) (type default) (color 0 0 0 0))
   )
-  (wire (pts (xy 184.15 144.78) (xy 184.15 146.05))
-    (stroke (width 0) (type default) (color 0 0 0 0))
-  )
   (wire (pts (xy 129.54 30.48) (xy 139.7 30.48))
     (stroke (width 0) (type default) (color 0 0 0 0))
@@
     (stroke (width 0) (type default) (color 0 0 0 0))
   )
-  (wire (pts (xy 172.72 138.43) (xy 181.61 138.43))
-    (stroke (width 0) (type default) (color 0 0 0 0))
-  )
   (wire (pts (xy 52.07 40.64) (xy 58.42 40.64))
     (stroke (width 0) (type default) (color 0 0 0 0))
@@
     (stroke (width 0) (type default) (color 0 0 0 0))
   )
-  (wire (pts (xy 181.61 135.89) (xy 181.61 138.43))
-    (stroke (width 0) (type default) (color 0 0 0 0))
-  )
   (wire (pts (xy 109.22 46.99) (xy 110.49 46.99))
     (stroke (width 0) (type default) (color 0 0 0 0))
@@
     (stroke (width 0) (type default) (color 0 0 0 0))
   )
-  (wire (pts (xy 179.07 146.05) (xy 184.15 146.05))
-    (stroke (width 0) (type default) (color 0 0 0 0))
-  )
   (polyline (pts (xy 15.24 21.59) (xy 15.24 144.78))
     (stroke (width 0) (type default) (color 0 0 0 0))
@@
     (stroke (width 0) (type default) (color 0 0 0 0))
   )
-  (wire (pts (xy 184.15 138.43) (xy 184.15 139.7))
-    (stroke (width 0) (type default) (color 0 0 0 0))
-  )
   (wire (pts (xy 36.83 87.63) (xy 43.18 87.63))
     (stroke (width 0) (type default) (color 0 0 0 0))
@@
   )
   (text "Flash Memory" (at 196.85 111.76 0)
-    (effects (font (size 1.27 1.27)) (justify left bottom))
-  )
-  (text "LDO" (at 123.19 157.48 0)
-    (effects (font (size 1.27 1.27)) (justify left bottom))
-  )
-  (text "Level Shifter Candidate:\nNLSX4302EBMUTCG\nC893527" (at 96.52 153.67 0)
     (effects (font (size 1.27 1.27)) (justify left bottom))
   )
@@
     )
   )
-  (global_label "VBUS" (shape input) (at 48.26 151.13 180) (fields_autoplaced)
-    (effects (font (size 1.27 1.27)) (justify right))
-    (property "Intersheet References" "${INTERSHEET_REFS}" (id 0) (at 40.9483 151.2094 0)
-      (effects (font (size 1.27 1.27)) (justify right) hide)
-    )
-  )
   (global_label "GPIO27{slash}ADC1" (shape tri_state) (at 109.22 115.57 0) (fields_autoplaced)
     (effects (font (size 1.27 1.27)) (justify left))
@@
     (property "Intersheet References" "${INTERSHEET_REFS}" (id 0) (at 118.5274 90.0906 0)
       (effects (font (size 1.27 1.27)) (justify left) hide)
-    )
-  )
-  (global_label "VBUS" (shape input) (at 180.34 135.89 180) (fields_autoplaced)
-    (effects (font (size 1.27 1.27)) (justify right))
-    (property "Intersheet References" "${INTERSHEET_REFS}" (id 0) (at 173.0283 135.9694 0)
-      (effects (font (size 1.27 1.27)) (justify right) hide)
     )
   )
@@
     (pin "2")
   )
-  (symbol (lib_id "Connector_Generic:Conn_01x01") (at 53.34 151.13 0) (unit 1)
-    (in_bom yes) (on_board yes)
-    (property "Reference" "J204" (id 0) (at 54.61 151.13 0)
-      (effects (font (size 1.27 1.27)) (justify left))
-    )
-    (property "Value" "5V" (id 1) (at 60.96 151.13 0)
-      (effects (font (size 1.27 1.27)) (justify left))
-    )
-    (property "Footprint" "Connector_PinSocket_2.54mm:PinSocket_1x01_P2.54mm_Vertical" (id 2) (at 53.34 151.13 0)
-      (effects (font (size 1.27 1.27)) hide)
-    )
-    (property "Datasheet" "~" (id 3) (at 53.34 151.13 0)
-      (effects (font (size 1.27 1.27)) hide)
-    )
-    (pin "1")
-  )
   (symbol (lib_id "Device:C_Small") (at 139.7 44.45 0) (unit 1)
     (in_bom yes) (on_board yes)
@@
     )
     (property "Datasheet" "" (id 3) (at 129.54 46.99 0)
-      (effects (font (size 1.27 1.27)) hide)
-    )
-    (pin "1")
-  )
-  (symbol (lib_id "Connector_Generic:Conn_01x01") (at 53.34 154.94 0) (unit 1)
-    (in_bom yes) (on_board yes)
-    (property "Reference" "J205" (id 0) (at 54.61 154.94 0)
-      (effects (font (size 1.27 1.27)) (justify left))
-    )
-    (property "Value" "TO BE DECIDED" (id 1) (at 60.96 154.94 0)
-      (effects (font (size 1.27 1.27)) (justify left))
-    )
-    (property "Footprint" "Connector_PinSocket_2.54mm:PinSocket_1x01_P2.54mm_Vertical" (id 2) (at 53.34 154.94 0)
-      (effects (font (size 1.27 1.27)) hide)
-    )
-    (property "Datasheet" "~" (id 3) (at 53.34 154.94 0)
       (effects (font (size 1.27 1.27)) hide)
     )
@@
     (pin "2")
   )
-  (symbol (lib_id "Connector_Generic:Conn_01x01") (at 53.34 158.75 0) (unit 1)
-    (in_bom yes) (on_board yes)
-    (property "Reference" "J206" (id 0) (at 54.61 158.75 0)
-      (effects (font (size 1.27 1.27)) (justify left))
-    )
-    (property "Value" "GND" (id 1) (at 60.96 158.75 0)
-      (effects (font (size 1.27 1.27)) (justify left))
-    )
-    (property "Footprint" "Connector_PinSocket_2.54mm:PinSocket_1x01_P2.54mm_Vertical" (id 2) (at 53.34 158.75 0)
-      (effects (font (size 1.27 1.27)) hide)
-    )
-    (property "Datasheet" "~" (id 3) (at 53.34 158.75 0)
-      (effects (font (size 1.27 1.27)) hide)
-    )
-    (pin "1")
-  )
-  (symbol (lib_id "Device:C_Small") (at 172.72 142.24 0) (unit 1)
-    (in_bom yes) (on_board yes)
-    (property "Reference" "C207" (id 0) (at 175.26 140.97 0)
-      (effects (font (size 1.27 1.27)) (justify left))
-    )
-    (property "Value" "220uF" (id 1) (at 175.26 143.51 0)
-      (effects (font (size 1.27 1.27)) (justify left))
-    )
-    (property "Footprint" "Capacitor_SMD:C_1210_3225Metric" (id 2) (at 172.72 142.24 0)
-      (effects (font (size 1.27 1.27)) hide)
-    )
-    (property "Datasheet" "~" (id 3) (at 172.72 142.24 0)
-      (effects (font (size 1.27 1.27)) hide)
-    )
-    (property "JLCPCB P/N" "C400951" (id 4) (at 172.72 142.24 0)
-      (effects (font (size 1.27 1.27)) hide)
-    )
-    (pin "1")
-    (pin "2")
-  )
   (symbol (lib_id "Device:C_Small") (at 29.21 43.18 0) (unit 1)
     (in_bom yes) (on_board yes)
@@
     (pin "1")
     (pin "2")
-  )
-  (symbol (lib_id "power:GND") (at 48.26 158.75 0) (unit 1)
-    (in_bom yes) (on_board yes) (fields_autoplaced)
-    (property "Reference" "#PWR0201" (id 0) (at 48.26 165.1 0)
-      (effects (font (size 1.27 1.27)) hide)
-    )
-    (property "Value" "GND" (id 1) (at 48.26 163.83 0))
-    (property "Footprint" "" (id 2) (at 48.26 158.75 0)
-      (effects (font (size 1.27 1.27)) hide)
-    )
-    (property "Datasheet" "" (id 3) (at 48.26 158.75 0)
-      (effects (font (size 1.27 1.27)) hide)
-    )
-    (pin "1")
   )
   (symbol (lib_id "power:GND") (at 119.38 35.56 0) (unit 1)
@@
     (pin "9")
   )
-  (symbol (lib_id "power:GND") (at 179.07 146.05 0) (unit 1)
-    (in_bom yes) (on_board yes)
-    (property "Reference" "#PWR0210" (id 0) (at 179.07 152.4 0)
-      (effects (font (size 1.27 1.27)) hide)
-    )
-    (property "Value" "GND" (id 1) (at 179.07 149.86 0))
-    (property "Footprint" "" (id 2) (at 179.07 146.05 0)
-      (effects (font (size 1.27 1.27)) hide)
-    )
-    (property "Datasheet" "" (id 3) (at 179.07 146.05 0)
-      (effects (font (size 1.27 1.27)) hide)
-    )
-    (pin "1")
-  )
   (symbol (lib_id "Memory_Flash:W25Q128JVS") (at 251.46 143.51 0) (unit 1)
     (in_bom yes) (on_board yes) (fields_autoplaced)
@@
     (pin "1")
   )
-  (symbol (lib_id "Device:C_Small") (at 184.15 142.24 0) (unit 1)
-    (in_bom yes) (on_board yes)
-    (property "Reference" "C209" (id 0) (at 186.69 140.97 0)
-      (effects (font (size 1.27 1.27)) (justify left))
-    )
-    (property "Value" "220uF" (id 1) (at 186.69 143.51 0)
-      (effects (font (size 1.27 1.27)) (justify left))
-    )
-    (property "Footprint" "Capacitor_SMD:C_1210_3225Metric" (id 2) (at 184.15 142.24 0)
-      (effects (font (size 1.27 1.27)) hide)
-    )
-    (property "Datasheet" "~" (id 3) (at 184.15 142.24 0)
-      (effects (font (size 1.27 1.27)) hide)
-    )
-    (property "JLCPCB P/N" "C400951" (id 4) (at 184.15 142.24 0)
-      (effects (font (size 1.27 1.27)) hide)
-    )
-    (pin "1")
-    (pin "2")
-  )
   (symbol (lib_id "power:GND") (at 48.26 190.5 0) (unit 1)
